Commit message: try tuning the feature tracker for better features

File: rviz/simple_car_model.urdf (robot description, URDF)
Before this commit: robot fourwheelrobot, 9 links, 8 joints
Links:
- removed link camera_link
- removed link imu_link
- added link cam0; visual box size=0.02 0.02 0.02
- added link imu0; visual box size=0.02 0.02 0.02
Joints:
- joint joint_camera: child camera_link -> cam0; parent imu_link -> imu0
- joint joint_imu: child imu_link -> imu0
